Commit message: URDF FIX

File: urdf/speeder_descriptionOLD2/robot.urdf (robot description, URDF)
Before this commit: robot droid, 14 links, 13 joints
Joints:
- joint base_leg_1: limit lower=-1.39626 upper=1.39626 effort=10 velocity=10 -> lower=-1.5707963268 upper=1.5707963268 effort=10 velocity=10
- joint first_leg_1: limit lower=-1.22173 upper=0.785398 effort=10 velocity=10 -> lower=-0.785398 upper=1.22173 effort=10 velocity=10; origin xyz=-0 0.005 -0.015 rpy=1.5708 -1.39626 -0 -> xyz=0 0.005 -0.015 rpy=1.5708 -0.959931 -0
- joint first_leg_2: limit lower=-1.22173 upper=0.785398 effort=10 velocity=10 -> lower=-0.785398 upper=1.22173 effort=10 velocity=10; origin xyz=-0 0.005 -0.015 rpy=1.5708 -1.39626 -0 -> xyz=0 0.005 -0.015 rpy=1.5708 -0.959931 -0
- joint first_leg_3: limit lower=-1.22173 upper=0.785398 effort=10 velocity=10 -> lower=-0.785398 upper=1.22173 effort=10 velocity=10; origin xyz=-0 0.005 -0.015 rpy=1.5708 -1.39626 -0 -> xyz=0 0.005 -0.015 rpy=1.5708 -0.959931 -0
- joint first_leg_4: limit lower=-1.22173 upper=0.785398 effort=10 velocity=10 -> lower=-0.785398 upper=1.22173 effort=10 velocity=10; origin xyz=0 0.005 -0.015 rpy=1.5708 -1.39626 -0 -> xyz=0 0.005 -0.015 rpy=1.5708 -0.959931 -0
- joint second_leg_1: limit lower=-1.5708 upper=1.13446 effort=10 velocity=10 -> lower=-1.13446 upper=1.5708 effort=10 velocity=10; origin xyz=-0 -0.05 0.010036 rpy=-3.14159 0 -1.8326 -> xyz=-0 -0.05 0.010036 rpy=-3.14159 0 -1.39626
- joint second_leg_2: limit lower=-1.5708 upper=1.13446 effort=10 velocity=10 -> lower=-1.13446 upper=1.5708 effort=10 velocity=10; origin xyz=-0 -0.05 0.010036 rpy=3.14159 0 -1.8326 -> xyz=-0 -0.05 0.010036 rpy=-3.14159 0 -1.39626
- joint second_leg_3: limit lower=-1.5708 upper=1.13446 effort=10 velocity=10 -> lower=-0.813125 upper=1.89214 effort=10 velocity=10; origin xyz=-0 -0.05 0.010036 rpy=3.14159 0 -1.8326 -> xyz=-0 -0.05 0.010036 rpy=3.14159 -0 -1.07492
- joint second_leg_4: limit lower=-1.5708 upper=1.13446 effort=10 velocity=10 -> lower=-1.13446 upper=1.5708 effort=10 velocity=10; origin xyz=-0 -0.05 0.010036 rpy=3.14159 0 -1.8326 -> xyz=-0 -0.05 0.010036 rpy=-3.14159 0 -1.39626
