Commit message: fix lower and upper limit of the urdf

File: urdf/speeder_descriptionOLD3/robot.urdf (robot description, URDF)
Before this commit: robot droid, 14 links, 13 joints
Joints:
- joint base_leg_1: limit lower=-1.5708 upper=1.5708 effort=10 velocity=10 -> lower=-1.39626 upper=1.39626 effort=10 velocity=10; origin xyz=-0.015 -0.0225 0.0025 rpy=-3.14159 0 -2.35619 -> xyz=-0.015 -0.0225 0.0025 rpy=-3.14159 -0 -2.35619
- joint first_leg_1: origin xyz=0 0.005 -0.015 rpy=1.5708 -1.39626 -0 -> xyz=-0 0.005 -0.015 rpy=1.5708 -1.39626 -0
- joint second_leg_1: origin xyz=-0 -0.05 0.010036 rpy=-3.14159 -0 -1.8326 -> xyz=-0 -0.05 0.010036 rpy=-3.14159 0 -1.8326
